Commit message: whatever

File: model1.urdf (robot description, URDF)
Before this commit: robot prosty_robot, 2 links, 1 joints
Joints:
- joint base_ramie: limit (none) -> lower=-1.5 upper=1.5 effort=30 velocity=1.0; origin xyz=0 0 0.05 rpy=0 0 0 -> xyz=0 0 0.025 rpy=0 0 0

Commit message: Ramie2

File: model1.urdf (robot description, URDF)
Before this commit: robot prosty_robot, 2 links, 1 joints
Links:
- added link ramie2_link, mass 0.5; collision box size=0.13 0.13 1; visual box size=0.13 0.13 1
- link ramie_link: geometry collision box size=0.13 0.13 1; visual box size=0.13 0.13 1
Joints:
- removed joint base_ramie
- added joint base_ramie_joint: type revolute, parent base_link, child ramie_link, origin xyz=0 0 0.025 rpy=0 0 0, axis 0 0 1, limit lower=-1.5 upper=1.5 effort=30 velocity=1.0
- added joint ramie_ramie2_joint: type revolute, parent ramie_link, child ramie2_link, origin xyz=0 0 1.0 rpy=0 0 0, axis 1 0 0, limit lower=-1.5 upper=1.5 effort=30 velocity=1.0

Commit message: Ramie3

File: model1.urdf (robot description, URDF)
Before this commit: robot prosty_robot, 3 links, 2 joints
Links:
- added link ramie3_link, mass 2.0; collision box size=0.1 0.1 0.5; visual box size=0.1 0.1 0.5
- link base_link: mass 2.0 -> 10.0
- link ramie2_link: mass 0.5 -> 4.0; geometry collision box size=0.1 0.1 0.6; visual box size=0.1 0.1 0.6
- link ramie_link: mass 0.5 -> 3.0; geometry collision box size=0.13 0.13 0.2; visual box size=0.1 0.1 0.2
Joints:
- added joint ramie2_ramie3_joint: type revolute, parent ramie2_link, child ramie3_link, origin xyz=0 0 0.6 rpy=-1 0 0, axis 1 0 0, limit lower=-2.5 upper=2.5 effort=100 velocity=2.0
- joint base_ramie_joint: limit lower=-1.5 upper=1.5 effort=30 velocity=1.0 -> lower=-2.9 upper=2.9 effort=150 velocity=2.0
- joint ramie_ramie2_joint: limit lower=-1.5 upper=1.5 effort=30 velocity=1.0 -> lower=-2.0 upper=2.0 effort=150 velocity=2.0; origin xyz=0 0 1.0 rpy=0 0 0 -> xyz=0 0 0.2 rpy=1 0 0

Commit message: Dodanie manipulatora w urdf

File: model1.urdf (robot description, URDF)
Before this commit: robot prosty_robot, 4 links, 3 joints
Links:
- added link manipulator_link, mass 0.2; collision sphere radius=0.08; visual sphere radius=0.08
Joints:
- added joint ramie3_manipulator_joint: type fixed, parent ramie3_link, child manipulator_link, origin xyz=0 0 0.5 rpy=0 0 0

Commit message: przesuniete napedy

File: model1.urdf (robot description, URDF)
Before this commit: robot prosty_robot, 5 links, 4 joints
Links:
- link ramie2_link: geometry collision box size=0.1 0.1 0.6; visual box size=0.14 0.14 0.6
- link ramie3_link: geometry collision box size=0.1 0.1 0.5; visual box size=0.1 0.1 0.5
- link ramie_link: geometry collision box size=0.2 0.2 0.4; visual box size=0.2 0.2 0.3
Joints:
- joint base_ramie_joint: limit lower=-2.9 upper=2.9 effort=150 velocity=2.0 -> lower=-2.618 upper=2.618 effort=150 velocity=2.0
- joint ramie2_ramie3_joint: limit lower=-2.5 upper=2.5 effort=100 velocity=2.0 -> lower=-2.3 upper=2.4 effort=100 velocity=2.0; origin xyz=0 0 0.6 rpy=-1 0 0 -> xyz=-0.14 0 0.6 rpy=0 0 0
- joint ramie_ramie2_joint: limit lower=-2.0 upper=2.0 effort=150 velocity=2.0 -> lower=-1.0 upper=1.75 effort=150 velocity=2.0; origin xyz=0 0 0.2 rpy=1 0 0 -> xyz=0.16 0 0.3 rpy=0 0 0

Commit message: Poprawione proporcje

File: model1.urdf (robot description, URDF)
Before this commit: robot prosty_robot, 5 links, 4 joints
Links:
- link base_link: mass 10.0 -> 20.0
- link ramie2_link: mass 4.0 -> 10.0
- link ramie3_link: mass 2.0 -> 5.0
- link ramie_link: mass 3.0 -> 8.0
Joints:
- joint base_ramie_joint: limit lower=-2.618 upper=2.618 effort=150 velocity=2.0 -> lower=-2.618 upper=2.618 effort=400 velocity=2.0
- joint ramie2_ramie3_joint: limit lower=-2.3 upper=2.4 effort=100 velocity=2.0 -> lower=-2.3 upper=2.4 effort=250 velocity=2.0
- joint ramie_ramie2_joint: limit lower=-1.0 upper=1.75 effort=150 velocity=2.0 -> lower=-1.0 upper=1.75 effort=400 velocity=2.0

Commit message: Poprawienie komentarzy i przejście na manipulator z samym visual

File: model1.urdf (robot description, URDF)
Before this commit: robot prosty_robot, 5 links, 4 joints
Links:
- link manipulator_link: mass 0.2 -> None; geometry visual sphere radius=0.08
